Commit message: Modifications for friction values & pick and place

File: robotiq/robotiq_description/urdf/robotiq_85_gripper.transmission.xacro (robot description, xacro)
@@ -6,5 +6,5 @@
       <joint name="${prefix}robotiq_85_left_knuckle_joint">
         <!-- <hardwareInterface>PositionJointInterface</hardwareInterface> -->
-        <hardwareInterface>kJointInterface</hardwareInterface>
+        <hardwareInterface>EffortJointInterface</hardwareInterface>
       </joint>
       <actuator name="${prefix}robotiq_85_left_knuckle_motor">

File: robotiq/robotiq_description/urdf/robotiq_85_gripper.urdf copy.xacro (robot description, xacro)
@@ -39,5 +39,5 @@
       <axis xyz="0 0 1"/>
       <origin rpy="0.0 0.0 0.0" xyz="0.05490451627 -0.03060114443 0.0"/>
-      <limit lower="-3.14" upper="3.14" velocity="50.0" effort="1000"/>
+      <limit lower="-3.14" upper="3.14" velocity="100.0" effort="1000"/>
       <mimic joint="${prefix}robotiq_85_left_knuckle_joint"/>
     </joint>
@@ -133,5 +133,5 @@
       <axis xyz="0 0 1"/>
       <origin xyz="0.06142 0.0127 0" rpy="${pi} 0.0 0.0" />
-      <limit lower="-3.14" upper="3.14" velocity="0.5" effort="3.0"/>
+      <limit lower="-3.14" upper="3.14" velocity="100.0" effort="1.5"/>
       <mimic joint="${prefix}robotiq_85_left_knuckle_joint" offset="0"/>
     </joint>
@@ -141,5 +141,5 @@
       <axis xyz="0 0 1"/>
       <origin xyz="0.06142 -0.0127 0" rpy="0 0 0"/>
-      <limit lower="-3.14" upper="3.14" velocity="50.0" effort="3.0"/>
+      <limit lower="-3.14" upper="3.14" velocity="100.0" effort="1.5"/>
       <mimic joint="${prefix}robotiq_85_left_knuckle_joint" offset="0"/>
     </joint>
@@ -240,6 +240,6 @@
       <kp>1000000.0</kp>
       <kd>1.0</kd>
-      <mu1>0.0001</mu1>
-      <mu2>0.0001</mu2>
+      <mu1>1.0</mu1>
+      <mu2>1.0</mu2>
       <minDepth>0.001</minDepth>
     </gazebo>
@@ -247,6 +247,6 @@
       <kp>1000000.0</kp>
       <kd>1.0</kd>
-      <mu1>0.0001</mu1>
-      <mu2>0.0001</mu2>
+      <mu1>1.0</mu1>
+      <mu2>1.0</mu2>
       <minDepth>0.001</minDepth>
     </gazebo>

File: universal_robot/ur_description/urdf/ur5_joint_limited_robot.urdf.xacro (robot description, xacro)
@@ -25,2 +25,3 @@
   </joint>
 </robot>
+<!-- wrist_2_lower_limit="${-pi}" wrist_2_upper_limit="${pi}" -->
