Commit message: Modified box & added mimic node

File: robotiq/robotiq_description/urdf/robotiq_85_gripper.urdf.xacro (robot description, xacro)
@@ -223,5 +223,5 @@
         </geometry>
       </visual>
-      <collision>
+      <collision name="robotiq_85_right_finger_tip_link_collision">
         <geometry>
           <mesh filename="package://robotiq_description/meshes/collision/robotiq_85_finger_tip_link.stl"/>
@@ -251,5 +251,32 @@
       <minDepth>0.001</minDepth>
     </gazebo>
+<!-- Bumper Plugin -->
+     <gazebo reference="${prefix}robotiq_85_left_finger_tip_link">
+        <sensor name="main_bumper" type="contact">
+            <selfCollide>true</selfCollide>
+            <alwaysOn>true</alwaysOn>
+            <updateRate>3.0</updateRate>
+            <material>Gazebo/Red</material>
+            <contact>
+                <collision>robotiq_85_right_finger_tip_link_collision</collision>
+            </contact>
+            <plugin name="bumper0_plugin" filename="libgazebo_ros_bumper.so">
+                <bumperTopicName>bumper_vals</bumperTopicName>
+                <frameName>robotiq_85_left_finger_tip_link</frameName>
+            </plugin>
+        </sensor>
+    </gazebo>
     <xacro:robotiq_85_gripper_transmission prefix="${prefix}" />
   </xacro:macro>
 </robot>
+<!-- libgazebo_ros_bumper -->
+<!-- Finger Contact Sensing -->
+    <!-- <gazebo reference="${prefix}robotiq_85_right_finger_tip_link">
+      <sensor name='my_contact' type='contact'>
+          <plugin name="my_plugin" filename="libcontact.so"/>
+              <contact>
+                <collision>robotiq_85_right_finger_tip_link_collision</collision>
+              </contact>
+            <update_rate> 5 </update_rate>
+            </sensor>
+      </gazebo> -->

Commit message: Manually added an object directly by creating a joint

File: robotiq/robotiq_description/urdf/robotiq_85_gripper.urdf.xacro (robot description, xacro)
@@ -200,13 +200,13 @@
 <!-- ____________________________________________________ -->
 <!-- Manually Added by AA for Mimicing an object intially in Hand -->
-    <!-- <joint name="${prefix}robotiq_85_object_grasp_joint" type="fixed">
+    <joint name="${prefix}robotiq_85_object_grasp_joint" type="fixed">
       <parent link="${prefix}robotiq_85_right_finger_tip_link"/>
       <child link="${prefix}robotiq_85_object_grasp_link"/>
       <axis xyz="0 0 1"/>
-      <origin rpy="0.0 0.0 0.0" xyz="0.04303959807 -0.03759940821  0.0"/> -->
-      <!-- <limit lower="-3.14" upper="3.14" velocity="100.0" effort="1.5"/> -->
-      <!-- <mimic joint="${prefix}robotiq_85_left_knuckle_joint" multiplier="-1"/> -->
-    <!-- </joint> -->
-<!-- Manually Added by AA for Mimicing an object intially in Hand
+      <origin rpy="0.0 0.0 0.0" xyz="0.04303959807 -0.03759940821  0.0"/>
+      <limit lower="-3.14" upper="3.14" velocity="100.0" effort="1.5"/>
+      <mimic joint="${prefix}robotiq_85_left_knuckle_joint" multiplier="-1"/>
+    </joint>
+<!-- Manually Added by AA for Mimicing an object intially in Hand -->
   <link name="${prefix}robotiq_85_object_grasp_link">
       <visual>
@@ -220,5 +220,5 @@
         </geometry>
       </collision>
-    </link>  -->
+    </link>
 <!-- ___________________________________________________ -->
     <link name="${prefix}robotiq_85_left_finger_tip_link">

Commit message: Added the correct initial position

File: robotiq/robotiq_description/urdf/robotiq_85_gripper.urdf.xacro (robot description, xacro)
@@ -200,5 +200,5 @@
 <!-- ____________________________________________________ -->
 <!-- Manually Added by AA for Mimicing an object intially in Hand -->
-    <joint name="${prefix}robotiq_85_object_grasp_joint" type="fixed">
+    <!-- <joint name="${prefix}robotiq_85_object_grasp_joint" type="fixed">
       <parent link="${prefix}robotiq_85_right_finger_tip_link"/>
       <child link="${prefix}robotiq_85_object_grasp_link"/>
@@ -207,7 +207,7 @@
       <limit lower="-3.14" upper="3.14" velocity="100.0" effort="1.5"/>
       <mimic joint="${prefix}robotiq_85_left_knuckle_joint" multiplier="-1"/>
-    </joint>
+    </joint> -->
 <!-- Manually Added by AA for Mimicing an object intially in Hand -->
-  <link name="${prefix}robotiq_85_object_grasp_link">
+  <!-- <link name="${prefix}robotiq_85_object_grasp_link">
       <visual>
         <geometry>
@@ -220,5 +220,5 @@
         </geometry>
       </collision>
-    </link>
+    </link>  -->
 <!-- ___________________________________________________ -->
     <link name="${prefix}robotiq_85_left_finger_tip_link">

File: universal_robot/ur_description/urdf/ur5.urdf.xacro (robot description, xacro)
@@ -98,5 +98,5 @@
       <parent link="${prefix}base_link" />
       <child link = "${prefix}shoulder_link" />
-      <origin xyz="0.0 0.0 ${shoulder_height}" rpy="0.0 0.0 0.0" />
+      <origin xyz="0.0 0.0 ${shoulder_height}" rpy="0.0 0.0 -1.57" />
       <axis xyz="0 0 1" />
       <xacro:unless value="${joint_limited}">
@@ -135,5 +135,5 @@
       <parent link="${prefix}shoulder_link" />
       <child link = "${prefix}upper_arm_link" />
-      <origin xyz="0.0 ${shoulder_offset} 0.0" rpy="0.0 1.36 0.0" />
+      <origin xyz="0.0 ${shoulder_offset} 0.0" rpy="0.0 0.0872665 0.0" />   <!--default values rpy="0.0 1.36 0.0-->
       <axis xyz="0 1 0" />
       <xacro:unless value="${joint_limited}">
@@ -172,5 +172,5 @@
       <parent link="${prefix}upper_arm_link" />
       <child link = "${prefix}forearm_link" />
-      <origin xyz="0.0 ${elbow_offset} ${upper_arm_length}" rpy="0.0 0.0 0.0" />
+      <origin xyz="0.0 ${elbow_offset} ${upper_arm_length}" rpy="0.0 1.57 0.0" />
       <axis xyz="0 1 0" />
       <xacro:unless value="${joint_limited}">
@@ -209,5 +209,5 @@
       <parent link="${prefix}forearm_link" />
       <child link = "${prefix}wrist_1_link" />
-      <origin xyz="0.0 0.0 ${forearm_length}" rpy="0.0 ${pi / 2.0} 0.0" />
+      <origin xyz="0.0 0.0 ${forearm_length}" rpy="0.0 0.174533 0.0" />   <!--rpy="0.0 0.26 0.0 working-->
       <axis xyz="0 1 0" />
       <xacro:unless value="${joint_limited}">
@@ -246,5 +246,5 @@
       <parent link="${prefix}wrist_1_link" />
       <child link = "${prefix}wrist_2_link" />
-      <origin xyz="0.0 ${wrist_1_length} 0.0" rpy="0.0 0.0 0.0" />
+      <origin xyz="0.0 ${wrist_1_length} 0.0" rpy="0.0 0.0 -1.48353" />  <!--Default rpy="0.0 0.0 -1.57"-->
       <axis xyz="0 0 1" />
       <xacro:unless value="${joint_limited}">

Commit message: attached object and working

File: robotiq/robotiq_description/urdf/robotiq_85_gripper.urdf.xacro (robot description, xacro)
@@ -200,5 +200,5 @@
 <!-- ____________________________________________________ -->
 <!-- Manually Added by AA for Mimicing an object intially in Hand -->
-    <!-- <joint name="${prefix}robotiq_85_object_grasp_joint" type="fixed">
+    <joint name="${prefix}robotiq_85_object_grasp_joint" type="fixed">
       <parent link="${prefix}robotiq_85_right_finger_tip_link"/>
       <child link="${prefix}robotiq_85_object_grasp_link"/>
@@ -206,8 +206,7 @@
       <origin rpy="0.0 0.0 0.0" xyz="0.04303959807 -0.03759940821  0.0"/>
       <limit lower="-3.14" upper="3.14" velocity="100.0" effort="1.5"/>
-      <mimic joint="${prefix}robotiq_85_left_knuckle_joint" multiplier="-1"/>
-    </joint> -->
+    </joint>
 <!-- Manually Added by AA for Mimicing an object intially in Hand -->
-  <!-- <link name="${prefix}robotiq_85_object_grasp_link">
+  <link name="${prefix}robotiq_85_object_grasp_link">
       <visual>
         <geometry>
@@ -220,5 +219,5 @@
         </geometry>
       </collision>
-    </link>  -->
+    </link>
 <!-- ___________________________________________________ -->
     <link name="${prefix}robotiq_85_left_finger_tip_link">
